File: Hekla.kicad_pcb (KiCad board)
At the start: 2 copper layers, 67 x 100 mm, 101 parts, among them J1 Thonkiconn, J10 Thonkiconn, J11 Thonkiconn, J12 Thonkiconn, J13 Thonkiconn, J14 Thonkiconn, J15 Conn_02x05_Odd_Even, J16 Conn_02x03_Odd_Even, J2 Thonkiconn, J3 Thonkiconn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

Commit message: First revision sent to production
Parts:
- D5, D6: value D -> US1M; footprint Diode_SMD:D_1812_4532Metric_Pad1.30x3.40mm_HandSolder -> Diode_SMD:D_SMA
- R17, R24: value 2.2k -> 2k2
- R2, R4: value 6.8k -> 6k8
- U2, U5: value LM4040DCK-10 -> LM4040DIM3-10.0/NOPB; footprint Package_TO_SOT_SMD:SOT-353_SC-70-5 -> Package_TO_SOT_SMD:SOT-23
- U4, U6, U7: value MCP6001-OT -> MCP6001T-E/OT
- U9: value IFX27001TFV50 -> AMS1117-5.0; footprint Package_TO_SOT_SMD:TO-252-3_TabPin2 -> Package_TO_SOT_SMD:SOT-223-3_TabPin2
- moved U5 58.7 mm to (119.6, 127.2), turned to 180 degrees
- moved C10 58.7 mm to (116.5, 127.3)
- moved R29 57.1 mm to (150.8, 138.0)
- moved U2 56.8 mm to (121.2, 142.8), turned to 270 degrees
- moved D6 56.8 mm to (118.5, 111.7), turned to 0 degrees
- moved R32 56.7 mm to (124.8, 90.9)
- moved C20 56.7 mm to (111.5, 112.2)
- moved C1 56.7 mm to (138.8, 117.9)
- moved C3 56.7 mm to (151.0, 118.5)
- moved D2 56.7 mm to (130.8, 155.0)
- moved D3 56.7 mm to (147.9, 155.0)
- moved JP2 56.7 mm to (167.8, 105.0)
- moved Q2 56.7 mm to (140.5, 75.8)
- moved Q3 56.7 mm to (128.5, 75.8)
- moved R37 56.7 mm to (133.8, 139.9)
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Connections:
- D6 pad 1: Net-(D6-Pad1) -> -12V
- D6 pad 2: -12V -> Net-(D6-Pad2)
- J15 pad 1: Net-(D6-Pad1) -> Net-(D6-Pad2)
- J15 pad 2: Net-(D6-Pad1) -> Net-(D6-Pad2)
- U2 pad 1: /-10Ref -> GND
- U2 pad 2: (no net) -> /-10Ref
- U2 pad 3: GND -> (no net)
- U5 pad 1: /10Ref -> +12V
- U5 pad 2: (no net) -> /10Ref
- U5 pad 3: +12V -> (no net)
Routing:
- net +5V: track 145.0 -> 128.6 mm
- net Net-(D6-Pad2): track 0.00 -> 14.6 mm
- net Net-(D6-Pad1): track 14.3 -> 0.00 mm
- net GND: track 31.9 -> 18.5 mm, vias 5 -> 333
- net +3V3: track 282.7 -> 293.7 mm
- net /10Ref: track 78.6 -> 83.7 mm
- net /SDA: track 44.7 -> 49.7 mm
- net /CVO2: track 28.5 -> 32.6 mm
- net /D5: track 45.8 -> 49.7 mm
- net -12V: track 69.9 -> 66.3 mm
- net /A3: track 37.3 -> 40.5 mm
- net /CVO1: track 56.6 -> 59.3 mm
- net +12V: track 56.0 -> 58.7 mm
- net /-10Ref: track 126.0 -> 127.7 mm
- net /A4: track 21.4 -> 20.1 mm
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- added copper zone on F.Cu, net GND
Other:
- board text added: "3V3"
- board text added: "GND"
- board text added: "MISO"
- board text added: "MOSI"
- board text added: "SCL"
- board text added: "Wiggle knobs and punch nazis!"
- board text removed: "Gate 1"
