File: Hekla.sch (KiCad schematic (older format))
At the start: 101 parts, among them J1 Thonkiconn, J10 Thonkiconn, J11 Thonkiconn, J12 Thonkiconn, J13 Thonkiconn, J14 Thonkiconn, J15 Conn_02x05_Odd_Even, J16 Conn_02x03_Odd_Even, J2 Thonkiconn, J3 Thonkiconn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

Commit message: First revision sent to production
Parts:
- removed D5, D6: D, Diode_SMD:D_1812_4532Metric_Pad1.30x3.40mm_HandSolder, symbol Device:D
- removed U2, U5: LM4040DCK-10, Package_TO_SOT_SMD:SOT-353_SC-70-5, symbol Reference_Voltage:LM4040DCK-10
- removed U9: IFX27001TFV50, Package_TO_SOT_SMD:TO-252-3_TabPin2, symbol Regulator_Linear:IFX27001TFV50
- added D5, D6: US1M, Diode_SMD:D_SMA, symbol Diode:US1M
- added U2, U5: LM4040DIM3-10.0/NOPB, Package_TO_SOT_SMD:SOT-23, symbol Reference_Voltage:LM4040DBZ-10
- added U9: AMS1117-5.0, Package_TO_SOT_SMD:SOT-223-3_TabPin2, symbol Regulator_Linear:AMS1117-5.0
- C1, C19, C2, C20: LCSC (none) -> C249452
- C10, C13, C14, C15, C16, C17, C18, C21, C3, C4, C7: LCSC (none) -> C14663
- C11, C12, C5, C6, C8, C9: LCSC (none) -> C1647
- Q1, Q2, Q3, Q4: LCSC (none) -> C20526
- R1, R3, R7, R8: LCSC (none) -> C25819
- R10, R15, R16, R9: LCSC (none) -> C25804
- R11, R12, R31, R32, R33, R34: LCSC (none) -> C21190
- R13, R14, R18, R20, R25, R27, R5, R6: LCSC (none) -> C25803
- R17, R24: value 2.2k -> 2k2; LCSC (none) -> C4190
- R19, R21, R26, R28, R36, R37, R38, R39: LCSC (none) -> C23192
- R2, R4: value 6.8k -> 6k8; LCSC (none) -> C23212
- R22, R23, R29, R30: LCSC (none) -> C23254
- R35: LCSC (none) -> C22775
- U1: LCSC (none) -> C6961
- U3: LCSC (none) -> C29429
- U4, U6, U7: value MCP6001-OT -> MCP6001T-E/OT; LCSC (none) -> C29429
- U8: LCSC (none) -> C7734
Connections:
- net +12V: now also D5.1 (K), U5.1 (K), U9.3 (VI)
- net +5V: now also U9.2 (VO)
- net -10Ref: now also U2.2 (A)
- net -12V: now also D6.1 (K)
- net 10Ref: now also U5.2 (A)
- net GND: now also U2.1 (K), U9.1 (GND)
- net at J15.1 (Pin_1), J15.2 (Pin_2): now also D6.2 (A)
- net at J15.10 (Pin_10), J15.9 (Pin_9): now also D5.2 (A)
Other:
- moved on the sheet: C7, R17
